Commit message: update for running example

File: Visualization/urdf/MiniCheetah/mini_cheetah_simple_correctedInertia.urdf (robot description, URDF)
Before this commit: robot mini_cheetah, 13 links, 12 joints
Links:
- added link foot_fl; collision sphere radius=0.0175; visual sphere radius=0.0175
- added link foot_fr; collision sphere radius=0.0175; visual sphere radius=0.0175
- added link foot_hl; collision sphere radius=0.0175; visual sphere radius=0.0175
- added link foot_hr; collision sphere radius=0.0175; visual sphere radius=0.0175
- link abduct_fl: geometry collision cylinder length=0.01 radius=0.0475; collision cylinder length=0.06 radius=0.0425
- link abduct_fr: geometry collision cylinder length=0.01 radius=0.0475; collision cylinder length=0.06 radius=0.0425
- link abduct_hl: geometry collision cylinder length=0.01 radius=0.0475; collision cylinder length=0.06 radius=0.0425
- link abduct_hr: geometry collision cylinder length=0.01 radius=0.0475; collision cylinder length=0.06 radius=0.0425
- link body: geometry collision box size=0.23 0.18 0.1; visual mesh filename=meshes/mini_body.obj
- link shank_fl: geometry collision cylinder length=0.15 radius=0.01; visual cylinder length=0.15 radius=0.01
- link shank_fr: geometry collision cylinder length=0.15 radius=0.01; visual cylinder length=0.15 radius=0.01
- link shank_hl: geometry collision cylinder length=0.15 radius=0.01; visual cylinder length=0.15 radius=0.01
- link shank_hr: geometry collision cylinder length=0.15 radius=0.01; visual cylinder length=0.15 radius=0.01
- link thigh_fl: geometry collision cylinder length=0.17 radius=0.015; visual cylinder length=0.17 radius=0.015
- link thigh_fr: geometry collision cylinder length=0.17 radius=0.015; visual cylinder length=0.17 radius=0.015
- link thigh_hl: geometry collision cylinder length=0.17 radius=0.015; visual cylinder length=0.17 radius=0.015
- link thigh_hr: geometry collision cylinder length=0.17 radius=0.015; visual cylinder length=0.17 radius=0.015
Joints:
- added joint fixed_shank_to_foot: type fixed, parent shank_fl, child foot_fl, origin xyz=0.0 0.0 -0.195 rpy=0.0 0.0 0.0
- added joint fixed_shank_to_foot_fr: type fixed, parent shank_fr, child foot_fr, origin xyz=0.0 0.0 -0.195 rpy=0.0 0.0 0.0
- added joint fixed_shank_to_foot_hl: type fixed, parent shank_hl, child foot_hl, origin xyz=0.0 0.0 -0.195 rpy=0.0 0.0 0.0
- added joint fixed_shank_to_foot_hr: type fixed, parent shank_hr, child foot_hr, origin xyz=0.0 0.0 -0.195 rpy=0.0 0.0 0.0
- joint abduct_fl_to_thigh_fl_j: axis 0 -1 0 -> 0 1 0; type continuous -> revolute
- joint abduct_fr_to_thigh_fr_j: axis 0 -1 0 -> 0 1 0; type continuous -> revolute
- joint abduct_hl_to_thigh_hl_j: axis 0 -1 0 -> 0 1 0; type continuous -> revolute
- joint abduct_hr_to_thigh_hr_j: axis 0 -1 0 -> 0 1 0; type continuous -> revolute
- joint thigh_fl_to_knee_fl_j: axis 0 -1 0 -> 0 1 0; type continuous -> revolute
- joint thigh_fr_to_knee_fr_j: axis 0 -1 0 -> 0 1 0; type continuous -> revolute
- joint thigh_hl_to_knee_hl_j: axis 0 -1 0 -> 0 1 0; type continuous -> revolute
- joint thigh_hr_to_knee_hr_j: axis 0 -1 0 -> 0 1 0; type continuous -> revolute
- joint torso_to_abduct_fl_j: type continuous -> revolute
- joint torso_to_abduct_fr_j: type continuous -> revolute
- joint torso_to_abduct_hl_j: type continuous -> revolute
- joint torso_to_abduct_hr_j: type continuous -> revolute
